File: Traffic_Light_Controller_guide.kicad_pcb (KiCad board)
At the start: 2 copper layers, 64 parts, among them J1 Conn_02x08_Odd_Even, J2 Conn_02x08_Odd_Even, J3 Conn_02x05_Odd_Even, J4 +5V, SW1 SW_Push, SW2 OVR, SW3 EN, U1 SM420561N, U2 SM420561N, U3 LM1117DT-3.3

Commit message: FINISH EXAM
Parts:
- added G***: LOGO, my_footprints:jinwoo, F.Cu at (153.5, 111.0)
- C3: footprint Capacitor_SMD:CP_Elec_6.3x3 -> Capacitor_SMD:CP_Elec_4x5.3
- C4: footprint Capacitor_SMD:CP_Elec_6.3x3 -> Capacitor_SMD:CP_Elec_6.3x5.8
- C5: footprint Capacitor_SMD:C_1206_3216Metric_Pad1.33x1.80mm_HandSolder -> LED_SMD:LED_1206_3216Metric_Pad1.42x1.75mm_HandSolder
- D1: value NSC_GRN -> GREEN; footprint Diode_SMD:D_1206_3216Metric_Pad1.42x1.75mm_HandSolder -> LED_THT:LED_D5.0mm
- D10, D9: footprint LED_SMD:LED_1206_3216Metric_Pad1.42x1.75mm_HandSolder -> LED_THT:LED_D5.0mm
- D2: value NSC_YLW -> YELLOW; footprint Diode_SMD:D_1206_3216Metric_Pad1.42x1.75mm_HandSolder -> LED_THT:LED_D5.0mm
- D3: value NSC_RED -> RED; footprint Diode_SMD:D_1206_3216Metric_Pad1.42x1.75mm_HandSolder -> LED_THT:LED_D5.0mm
- D4: value EWC_GRN -> GREEN; footprint Diode_SMD:D_1206_3216Metric_Pad1.42x1.75mm_HandSolder -> LED_THT:LED_D5.0mm
- D5: value EWC_YLW -> YELLOW; footprint Diode_SMD:D_1206_3216Metric_Pad1.42x1.75mm_HandSolder -> LED_THT:LED_D5.0mm
- D6: value EWC_RED -> RED; footprint Diode_SMD:D_1206_3216Metric_Pad1.42x1.75mm_HandSolder -> LED_THT:LED_D5.0mm
- D7: value LED -> GREEN; footprint LED_SMD:LED_1206_3216Metric_Pad1.42x1.75mm_HandSolder -> LED_THT:LED_D5.0mm
- D8: value LED -> RED; footprint LED_SMD:LED_1206_3216Metric_Pad1.42x1.75mm_HandSolder -> LED_THT:LED_D5.0mm
- R1, R10, R14, R15, R17, R18, R19, R2, R20, R21, R22, R23, R24, R25, R26, R3, R4, R5, R6, R7, R8, R9: value 130 -> 130R
- SW1: value SW_Push -> RST
- U3: footprint Package_TO_SOT_SMD:TO-252-3_TabPin2 -> Package_TO_SOT_SMD:SOT-223-3_TabPin2
- moved D8 238.0 mm to (164.5, 65.5), turned to 180 degrees
- moved D7 237.2 mm to (164.5, 55.5), turned to 180 degrees
- moved R24 229.0 mm to (172.0, 65.5), turned to 180 degrees
- moved R23 227.9 mm to (172.0, 55.5), turned to 180 degrees
- moved R28 226.8 mm to (162.5, 93.0)
- moved R3 223.9 mm to (150.5, 74.0), turned to 90 degrees
- moved R8 223.9 mm to (154.5, 74.0), turned to 90 degrees
- moved R27 222.7 mm to (162.5, 89.0)
- moved R2 222.5 mm to (154.5, 46.5), turned to -90 degrees
- moved D12 219.5 mm to (162.5, 97.0), turned to 180 degrees
- moved R4 219.2 mm to (146.5, 74.0), turned to 90 degrees
- moved R1 219.2 mm to (150.5, 46.5), turned to -90 degrees
- moved R5 214.5 mm to (142.5, 74.0), turned to 90 degrees
- moved H4 214.0 mm to (173.0, 117.0)
- moved SW1 213.2 mm to (154.5, 97.5)
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Connections:
- C5 pad 2: unconnected-(C5-Pad2) -> GND
- R31 pad 2: unconnected-(R31-Pad2) -> /+3.3V
Routing:
- net GND: track 0.00 -> 450.3 mm, vias 0 -> 4
- net /+3.3V: track 0.00 -> 272.5 mm, vias 0 -> 4
- net /EN: track 0.00 -> 159.6 mm
- net /OVR: track 0.00 -> 137.0 mm, vias 0 -> 2
- net /RST: track 0.00 -> 136.2 mm, vias 0 -> 2
- net /NS_HEX_A: track 0.00 -> 118.9 mm
- net /NS_HEX_B: track 0.00 -> 107.3 mm
- net /+5V: track 0.00 -> 83.9 mm
- net /EW_HEX_D: track 0.00 -> 75.1 mm
- net /NSP_RED: track 0.00 -> 75.1 mm
- net /NSP_GRN: track 0.00 -> 73.9 mm
- net /EW_HEX_C: track 0.00 -> 69.7 mm
- net /NS_HEX_DP: track 0.00 -> 68.1 mm, vias 0 -> 1
- net /NSC_GRN: track 0.00 -> 67.1 mm, vias 0 -> 2
- net /EW_HEX_E: track 0.00 -> 66.1 mm, vias 0 -> 1
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Other:
- board outline added: 125.5 x 83 mm
- board text added: "+3V3"
- board text added: "+5V"
- board text added: "A"
- board text added: "B"
- board text added: "C"
- board text added: "CAR"
- board text added: "D"
- board text added: "DP"
- board text added: "E"
- board text added: "E-W"
- board text added: "EAST-WEST TRAFFIC LIGHTS"
- board text added: "EN"
- board text added: "ENABLE"
- board text added: "EW CONNECTOR"
- board text added: "F"
- board text added: "FRANZ LOUIS G. VIGILAR 17 APRIL, 2026 Computer Engineering Technology Department Technological University of the Philippines Visayas"
- board text added: "G"
- board text added: "GND"
- board text added: "N-S"
- board text added: "NORTH-SOUTH TRAFFIC LIGHTS"
- board text added: "NS CONNECTOR"
- board text added: "OVERRIDE"
- board text added: "OVR"
- board text added: "PED"
- board text added: "R"
- board text added: "RESET"
- board text added: "RST"
- board text added: "Traffic Light Controller board for Finite State Machine (FSM) demo. It manages traffic flow for two perpendicular roads: North-South (NS) and East-West (EW)."
- board text added: "Y"

Commit message: Finish exam
Routing:
- net /OVR: track 137.0 -> 134.7 mm

Commit message: update pcb
Parts:
- R11, R12, R13, R16: value 130 -> 130R
